Commit message: Tutorial w28: tf, remap

File: src/my_r2d2/urdf/new.rd2d.xacro (robot description, xacro)
@@ -1,4 +1,4 @@
 <?xml version="1.0"?>
-<robot name="r2d2" xmlns:xacro="http://ros.org/wiki/xacro">
+<robot name="macroed" xmlns:xacro="http://ros.org/wiki/xacro">
   <xacro:property name="width" value=".2" />
   <xacro:property name="leglen" value=".6" />
@@ -213,10 +213,3 @@
     <origin xyz="${.707*width+0.04} 0 ${.707*width}"/>
   </joint>
-  <link name="base_footprint">
-  </link>
-  <joint name="base_footprint_link" type="fixed">
-    <parent link="base_footprint"/>
-    <child link="base_link"/>
-    <origin xyz="0 0 ${bodylen/2 + wheeldiam + 0.1}"/>
-  </joint>
 </robot>

File: src/my_r2d2/urdf/old.r2d2.urdf.xacro (robot description, xacro)
@@ -1,4 +1,4 @@
 <?xml version="1.0"?>
-<robot name="r2d2" xmlns:xacro="http://ros.org/wiki/xacro">
+<robot name="macroed" xmlns:xacro="http://ros.org/wiki/xacro">
   <xacro:property name="width" value=".2" />
   <xacro:property name="leglen" value=".6" />
