Commit message: "GR5 is in self-collision"

File: src/dual_manipulator_support/urdf/dual_manip.urdf (robot description, URDF)
Before this commit: robot dual_manip, 21 links, 20 joints
Links:
- removed link right_link_b
- removed link right_link_e
- removed link right_link_l
- removed link right_link_r
- removed link right_link_s
- removed link right_link_t
- removed link right_link_u
- added link right_ee_link; collision box size=0.01 0.01 0.01
- added link right_forearm_link, mass 2.275; collision mesh filename=package://ur_description/meshes/ur5/collision/forearm.stl; visual mesh filename=package://ur_description/meshes/ur5/visual/forearm.dae
- added link right_shoulder_link, mass 3.7; collision mesh filename=package://ur_description/meshes/ur5/collision/shoulder.stl; visual mesh filename=package://ur_description/meshes/ur5/visual/shoulder.dae
- added link right_upper_arm_link, mass 8.393; collision mesh filename=package://ur_description/meshes/ur5/collision/upperarm.stl; visual mesh filename=package://ur_description/meshes/ur5/visual/upperarm.dae
- added link right_wrist_1_link, mass 1.219; collision mesh filename=package://ur_description/meshes/ur5/collision/wrist1.stl; visual mesh filename=package://ur_description/meshes/ur5/visual/wrist1.dae
- added link right_wrist_2_link, mass 1.219; collision mesh filename=package://ur_description/meshes/ur5/collision/wrist2.stl; visual mesh filename=package://ur_description/meshes/ur5/visual/wrist2.dae
- added link right_wrist_3_link, mass 0.1879; collision mesh filename=package://ur_description/meshes/ur5/collision/wrist3.stl; visual mesh filename=package://ur_description/meshes/ur5/visual/wrist3.dae
- link right_base_link: mass None -> 4.0; geometry collision mesh filename=package://ur_description/meshes/ur5/collision/base.stl; visual mesh filename=package://ur_description/meshes/ur5/visual/base.dae
Joints:
- removed joint right_joint_b
- removed joint right_joint_e
- removed joint right_joint_l
- removed joint right_joint_r
- removed joint right_joint_s
- removed joint right_joint_t
- removed joint right_joint_u
- removed joint right_link_l-base
- removed joint right_link_t-tool0
- added joint right_base_link-base_fixed_joint: type fixed, parent right_base_link, child right_base, origin xyz=0 0 0 rpy=0 0 -3.14159265
- added joint right_ee_fixed_joint: type fixed, parent right_wrist_3_link, child right_ee_link, origin xyz=0.0 0.0823 0.0 rpy=0.0 0.0 1.570796325
- added joint right_elbow_joint: type revolute, parent right_upper_arm_link, child right_forearm_link, origin xyz=0.0 -0.1197 0.425 rpy=0.0 0.0 0.0, axis 0 1 0, limit lower=-6.2831853 upper=6.2831853 effort=150.0 velocity=3.15
- added joint right_shoulder_lift_joint: type revolute, parent right_shoulder_link, child right_upper_arm_link, origin xyz=0.0 0.13585 0.0 rpy=0.0 1.570796325 0.0, axis 0 1 0, limit lower=-6.2831853 upper=6.2831853 effort=150.0 velocity=3.15
- added joint right_shoulder_pan_joint: type revolute, parent right_base_link, child right_shoulder_link, origin xyz=0.0 0.0 0.089159 rpy=0.0 0.0 0.0, axis 0 0 1, limit lower=-6.2831853 upper=6.2831853 effort=150.0 velocity=3.15
- added joint right_wrist_1_joint: type revolute, parent right_forearm_link, child right_wrist_1_link, origin xyz=0.0 0.0 0.39225 rpy=0.0 1.570796325 0.0, axis 0 1 0, limit lower=-6.2831853 upper=6.2831853 effort=28.0 velocity=3.2
- added joint right_wrist_2_joint: type revolute, parent right_wrist_1_link, child right_wrist_2_link, origin xyz=0.0 0.093 0.0 rpy=0.0 0.0 0.0, axis 0 0 1, limit lower=-6.2831853 upper=6.2831853 effort=28.0 velocity=3.2
- added joint right_wrist_3_joint: type revolute, parent right_wrist_2_link, child right_wrist_3_link, origin xyz=0.0 0.0 0.09465 rpy=0.0 0.0 0.0, axis 0 1 0, limit lower=-6.2831853 upper=6.2831853 effort=28.0 velocity=3.2
- added joint right_wrist_3_link-tool0_fixed_joint: type fixed, parent right_wrist_3_link, child right_tool0, origin xyz=0 0.0823 0 rpy=-1.570796325 0 0

File: src/dual_manipulator_support/urdf/dual_manip.xacro (robot description, xacro)
@@ -5,5 +5,10 @@
 	<xacro:include filename="$(find motoman_sia5d_support)/urdf/sia5d_macro.xacro"/>
 	<xacro:motoman_sia5d prefix="left_"/>
-	<xacro:motoman_sia5d prefix="right_"/>
+	  <!-- common stuff -->
+  	<xacro:include filename="$(find ur_description)/urdf/common.gazebo.xacro" />
+  <!-- ur5 -->
+  	<xacro:include filename="$(find ur_description)/urdf/ur5.urdf.xacro" />
+  <!-- arm -->
+  	<xacro:ur5_robot prefix="right_" joint_limited="false"/>
 	<link name="base_link">
 		<visual>
